Commit message: Initial map my world

File: src/my_robot/urdf/my_robot.xacro (robot description, xacro)
@@ -107,5 +107,5 @@
         <dynamics damping="1.0" friction="1.0"/>
     </joint>
-    <link name='camera'>
+    <link name='camera_link'>
         <box_inertia m="0.1" x="0.05" y="0.05" z="0.05"/>
         <inertial>
@@ -114,5 +114,5 @@
             <inertia ixx="1e-6" ixy="0" ixz="0" iyy="1e-6" iyz="0" izz="1e-6" />
         </inertial>
-        <collision name='collision'>
+        <collision name='camera_collision'>
             <origin xyz="0 0 0" rpy="0 0 0"/>
             <geometry>
@@ -120,5 +120,5 @@
             </geometry>
         </collision>
-        <visual name='right_wheel_visual'>
+        <visual name='camera_visual'>
             <origin xyz="0 0 0" rpy="0 0 0"/>
             <geometry>
@@ -127,7 +127,14 @@
         </visual>
     </link>
+    <joint name="camera_optical_joint" type="fixed">
+        <origin xyz="0 0 0" rpy="-1.5707 0 -1.5707"/>
+        <parent link="camera_link"/>
+        <child link="camera_link_optical"/>
+    </joint>
+    <link name="camera_link_optical">
+    </link>
     <joint type="fixed" name="camera_joint">
         <origin xyz="0.2 0 0" rpy="0 0 0"/>
-        <child link="camera"/>
+        <child link="camera_link"/>
         <parent link="chassis"/>
         <axis xyz="0 1 0"/>
